File: hardware/kicad/analog_in.kicad_sch (KiCad schematic)
At the start: 66 parts, among them J10 AI4: +24V / IN / GND, J11 AI5: +24V / IN / GND, J12 AI6: +24V / IN / GND, J7 AI1: +24V / IN / GND, J8 AI2: +24V / IN / GND, J9 AI3: +24V / IN / GND, U3 ADS1115IDGS, U4 ADS1115IDGS

Commit message: hardware: Rev 0.2 – ESP32-S3 (Steuerung) + M5Stack Stamp-P4 (App/HMI) statt CM5
CM5 entfernt. Neu: ESP32-S3-WROOM-1 für Regelung/I/O/V20, Stamp-P4 mit
LAN8720A-Ethernet und 7"-MIPI-DSI-Touch (FPC 15p), UART-Link mit Reset/Boot-
Steuerung des S3 durch den P4, 5V->3,3V-Wandler, USB-Werkbankversorgung.
I/O-Blätter unverändert. Netzliste geprüft (180 Netze, 0 Fehler).

Co-Authored-By: Claude Opus 5.5 <noreply@anthropic.com>
Claude-Session: https://claude.ai/code/session_019gH4tfEhDrFu8dTGZD88nH
Parts:
- removed C22, C23, C24, C25, C26, C27: 10nF, Capacitor_SMD:C_0603_1608Metric, symbol Device:C
- removed C28, C29, C30, C31: 100nF, Capacitor_SMD:C_0603_1608Metric, symbol Device:C
- removed D5: SMAJ26A, Diode_SMD:D_SMA, symbol Diode:SMAJ26A
- removed F2: 50mA hold, Fuse:Fuse_1206_3216Metric, symbol Device:Polyfuse
- removed J7: AI1: +24V / IN / GND, TerminalBlock_Phoenix:TerminalBlock_Phoenix_PT-1,5-3-3.5-H_1x03_P3.50mm_Horizontal, symbol Connector:Screw_Terminal_01x03
- removed JP7: 4-20mA, Connector_PinHeader_2.54mm:PinHeader_1x02_P2.54mm_Vertical, symbol Jumper:Jumper_2_Open
- removed R20, R23, R26, R29, R32: 150 0.1% 1W, Resistor_SMD:R_2512_6332Metric, symbol Device:R
- removed R21, R24, R27, R30, R33: 22k 0.1%, Resistor_SMD:R_0603_1608Metric, symbol Device:R
- removed R22, R25, R28, R31, R34: 10k 0.1%, Resistor_SMD:R_0603_1608Metric, symbol Device:R
- removed U3, U4: ADS1115IDGS, Package_SO:TSSOP-10_3x3mm_P0.5mm, symbol Analog_ADC:ADS1115IDGS
- added C35, C36, C37, C38, C39, C40: 10nF, Capacitor_SMD:C_0603_1608Metric, symbol Device:C
- added C41, C42, C43, C44: 100nF, Capacitor_SMD:C_0603_1608Metric, symbol Device:C
- added D11: SMAJ26A, Diode_SMD:D_SMA, symbol Diode:SMAJ26A
- added F14: 50mA hold, Fuse:Fuse_1206_3216Metric, symbol Device:Polyfuse
- added J13: AI6: +24V / IN / GND, TerminalBlock_Phoenix:TerminalBlock_Phoenix_PT-1,5-3-3.5-H_1x03_P3.50mm_Horizontal, symbol Connector:Screw_Terminal_01x03
- added JP1: 4-20mA, Connector_PinHeader_2.54mm:PinHeader_1x02_P2.54mm_Vertical, symbol Jumper:Jumper_2_Open
- added R44, R47, R50: 150 0.1% 1W, Resistor_SMD:R_2512_6332Metric, symbol Device:R
- added R45, R48, R51: 22k 0.1%, Resistor_SMD:R_0603_1608Metric, symbol Device:R
- added R46, R49, R52: 10k 0.1%, Resistor_SMD:R_0603_1608Metric, symbol Device:R
- added R53: 100k 1%, Resistor_SMD:R_0603_1608Metric, symbol Device:R
- added R54, R55, R56: 10k 1%, Resistor_SMD:R_0603_1608Metric, symbol Device:R
- added R57, R58: 10k, Resistor_SMD:R_0603_1608Metric, symbol Device:R
- added U7, U8: ADS1115IDGS, Package_SO:TSSOP-10_3x3mm_P0.5mm, symbol Analog_ADC:ADS1115IDGS
- J10: value AI4: +24V / IN / GND -> AI3: +24V / IN / GND
- J11: value AI5: +24V / IN / GND -> AI4: +24V / IN / GND
- J12: value AI6: +24V / IN / GND -> AI5: +24V / IN / GND
- J8: value AI2: +24V / IN / GND -> AI1: +24V / IN / GND
- J9: value AI3: +24V / IN / GND -> AI2: +24V / IN / GND
- R38: value 100k 1% -> 150 0.1% 1W; footprint Resistor_SMD:R_0603_1608Metric -> Resistor_SMD:R_2512_6332Metric
- R39: value 10k 1% -> 22k 0.1%
- R40: value 10k 1% -> 10k 0.1%
- R41: value 10k 1% -> 150 0.1% 1W; footprint Resistor_SMD:R_0603_1608Metric -> Resistor_SMD:R_2512_6332Metric
- R42: value 10k -> 22k 0.1%
- R43: value 10k -> 10k 0.1%
Connections:
- net +24V: now also F11.1, F13.1, F3.1, F5.1, F7.1, F9.1, R53.1; no longer F10.1, F12.1, F4.1, F6.1, F8.1, R38.1
- net +3V3: now also C43.1, C44.1, R57.1, R58.1, U7.8 (VDD), U8.1 (ADDR), U8.8 (VDD); no longer R42.1, R43.1
- net +5V: now also R55.1; no longer R40.1
- net ADC1_ALERT: now also R57.2, U7.2 (ALERT/RDY); no longer R42.2
- net ADC2_ALERT: now also R58.2, U8.2 (ALERT/RDY); no longer R43.2
- net AI1_ADC: now also R36.2, R37.1, C35.1, U7.4 (AIN0)
- net AI1_IN: now also D6.1 (A1), F4.1, J8.2 (Pin_2); no longer F3.1
- net AI1_NODE: now also F4.2, R36.1, JP1.1 (A); no longer F3.2, JP2.1 (A)
- net AI1_PWR: now also F3.2, J8.1 (Pin_1)
- net AI1_SH: now also R35.1, JP1.2 (B); no longer JP2.2 (B)
- net AI2_ADC: now also R39.2, R40.1, C36.1, U7.5 (AIN1)
- net AI2_IN: now also D7.1 (A1), F6.1, J9.2 (Pin_2); no longer D6.1 (A1), F5.1, J8.2 (Pin_2)
- net AI2_NODE: now also F6.2, JP2.1 (A), R39.1; no longer F5.2, JP3.1 (A)
- net AI2_PWR: now also F5.2, J9.1 (Pin_1); no longer F4.2, J8.1 (Pin_1)
- net AI2_SH: now also JP2.2 (B), R38.1; no longer JP3.2 (B)
- net AI3_ADC: now also R42.2, R43.1, C37.1, U7.6 (AIN2)
- net AI3_IN: now also D8.1 (A1), F8.1, J10.2 (Pin_2); no longer D7.1 (A1), F7.1, J9.2 (Pin_2)
- net AI3_NODE: now also F8.2, JP3.1 (A), R42.1; no longer F7.2, JP4.1 (A)
- net AI3_PWR: now also F7.2, J10.1 (Pin_1); no longer F6.2, J9.1 (Pin_1)
- net AI3_SH: now also JP3.2 (B), R41.1; no longer JP4.2 (B)
- net AI4_ADC: now also C38.1, R45.2, R46.1, U7.7 (AIN3)
- net AI4_IN: now also D9.1 (A1), F10.1, J11.2 (Pin_2); no longer D8.1 (A1), F9.1, J10.2 (Pin_2)
- net AI4_NODE: now also F10.2, JP4.1 (A), R45.1; no longer F9.2, JP5.1 (A)
- net AI4_PWR: now also F9.2, J11.1 (Pin_1); no longer F8.2, J10.1 (Pin_1)
- net AI4_SH: now also JP4.2 (B), R44.1; no longer JP5.2 (B)
- net AI5_ADC: now also C39.1, R48.2, R49.1, U8.4 (AIN0)
- net AI5_IN: now also D10.1 (A1), F12.1, J12.2 (Pin_2); no longer D9.1 (A1), F11.1, J11.2 (Pin_2)
- net AI5_NODE: now also F12.2, JP5.1 (A), R48.1; no longer F11.2, JP6.1 (A)
- net AI5_PWR: now also F11.2, J12.1 (Pin_1); no longer F10.2, J11.1 (Pin_1)
- net AI5_SH: now also JP5.2 (B), R47.1; no longer JP6.2 (B)
- net AI6_ADC: now also C40.1, R51.2, R52.1, U8.5 (AIN1); no longer R36.2, R37.1
- net AI6_IN: now also D11.1 (A1), F14.1, J13.2 (Pin_2); no longer D10.1 (A1), F13.1, J12.2 (Pin_2)
- net AI6_NODE: now also JP6.1 (A), F14.2, R51.1; no longer F13.2, R36.1
- net AI6_PWR: now also F13.2, J13.1 (Pin_1); no longer F12.2, J12.1 (Pin_1)
- net AI6_SH: now also JP6.2 (B), R50.1; no longer R35.1
- net GND: now also R38.2, R40.2, R43.2, C35.2, C36.2, C37.2, C38.2, C39.2, C40.2, C41.2, C42.2, C43.2, C44.2, D11.2 (A2), J13.3 (Pin_3), R44.2, R46.2, R47.2, R49.2, R50.2, R52.2, R54.2, R56.2, U7.1 (ADDR), U7.3 (GND), U8.3 (GND); no longer R39.2
- net I2C_SCL: now also U7.10 (SCL), U8.10 (SCL)
- net I2C_SDA: now also U7.9 (SDA), U8.9 (SDA)
- net MON_24V: now also C41.1, R53.2, R54.1, U8.6 (AIN2); no longer R38.2, R39.1
- net MON_5V: now also C42.1, R55.2, R56.1, U8.7 (AIN3); no longer R40.2, R41.1

Commit message: hardware: Schaltplan im Block-Stil wie pool-pcb
Neuer Generator tools/schblock.py: gestrichelte Funktionsblöcke mit Titel und
Notizen, echte Drähte (eigener Router), Power-Symbole am Pin bzw. als Schiene,
Global-Labels nur an Blockgrenzen. Netzliste weiterhin gegen die deklarierte
Absicht geprüft (180 Netze, 0 Fehler), PWR_FLAGs ergänzt.

Co-Authored-By: Claude Opus 5.5 <noreply@anthropic.com>
Claude-Session: https://claude.ai/code/session_019gH4tfEhDrFu8dTGZD88nH
Parts:
- removed C44: 100nF, Capacitor_SMD:C_0603_1608Metric, symbol Device:C
- added C34: 10n, Capacitor_SMD:C_0603_1608Metric, symbol Device:C
- C35, C36, C37, C38, C39: value 10nF -> 10n
- C40: value 10nF -> 100nF
- C42, C43: value 100nF -> 100n
- F10, F11, F12, F13, F14, F3, F4, F5, F6, F7, F8, F9: value 50mA hold -> 50mA
- J10: value AI3: +24V / IN / GND -> AI3
- J11: value AI4: +24V / IN / GND -> AI4
- J12: value AI5: +24V / IN / GND -> AI5
- J13: value AI6: +24V / IN / GND -> AI6
- J8: value AI1: +24V / IN / GND -> AI1
- J9: value AI2: +24V / IN / GND -> AI2
- R53: value 100k 1% -> 10k
- R54: value 10k 1% -> 10k
- R55: value 10k 1% -> 100k 1%
- R57, R58: value 10k -> 10k 1%
Connections:
- net +24V: now also R55.1; no longer R53.1
- net +3V3: now also C40.1, C41.1, R53.1, R54.1; no longer C43.1, R57.1, R58.1
- net +5V: now also R57.1; no longer R55.1
- net ADC1_ALERT: now also R53.2; no longer R57.2
- net ADC2_ALERT: now also R54.2; no longer R58.2
- net AI1_ADC: now also C34.1; no longer C35.1
- net AI2_ADC: now also C35.1; no longer C36.1
- net AI3_ADC: now also C36.1; no longer C37.1
- net AI4_ADC: now also C37.1; no longer C38.1
- net AI5_ADC: now also C38.1; no longer C39.1
- net AI6_ADC: now also C39.1; no longer C40.1
- net GND: now also R58.2, C34.2; no longer R54.2
- net MON_24V: now also C42.1, R55.2, R56.1; no longer C41.1, R53.2, R54.1
- net MON_5V: now also C43.1, R57.2, R58.1; no longer C42.1, R55.2, R56.1
- net AI1_IN: no longer names the net of D6.1 (A1), F4.1, J8.2 (Pin_2)
- net AI1_NODE: no longer names the net of F4.2, JP1.1 (A), R36.1
- net AI1_PWR: no longer names the net of F3.2, J8.1 (Pin_1)
- net AI1_SH: no longer names the net of JP1.2 (B), R35.1
- net AI2_IN: no longer names the net of D7.1 (A1), F6.1, J9.2 (Pin_2)
- net AI2_NODE: no longer names the net of F6.2, JP2.1 (A), R39.1
- net AI2_PWR: no longer names the net of F5.2, J9.1 (Pin_1)
- net AI2_SH: no longer names the net of JP2.2 (B), R38.1
- net AI3_IN: no longer names the net of D8.1 (A1), F8.1, J10.2 (Pin_2)
- net AI3_NODE: no longer names the net of F8.2, JP3.1 (A), R42.1
- net AI3_PWR: no longer names the net of F7.2, J10.1 (Pin_1)
- net AI3_SH: no longer names the net of JP3.2 (B), R41.1
- net AI4_IN: no longer names the net of D9.1 (A1), F10.1, J11.2 (Pin_2)
- net AI4_NODE: no longer names the net of F10.2, JP4.1 (A), R45.1
- net AI4_PWR: no longer names the net of F9.2, J11.1 (Pin_1)
- net AI4_SH: no longer names the net of JP4.2 (B), R44.1
- net AI5_IN: no longer names the net of D10.1 (A1), F12.1, J12.2 (Pin_2)
- net AI5_NODE: no longer names the net of F12.2, JP5.1 (A), R48.1
- net AI5_PWR: no longer names the net of F11.2, J12.1 (Pin_1)
- net AI5_SH: no longer names the net of JP5.2 (B), R47.1
- net AI6_IN: no longer names the net of D11.1 (A1), F14.1, J13.2 (Pin_2)
- net AI6_NODE: no longer names the net of F14.2, JP6.1 (A), R51.1
- net AI6_PWR: no longer names the net of F13.2, J13.1 (Pin_1)
- net AI6_SH: no longer names the net of JP6.2 (B), R50.1
Other:
- note added: "ADC ADS1115 × 2 (I²C 0x48 / 0x49)"
- note added: "ADC1: AI1–AI4. ADC2: AI5, AI6, 24-V- und 5-V-Überwachung. 4–20 mA: PGA ±1,024 V (20 mA → 0,9375 V). 0–10 V: PGA ±4,096 V (10 V → 3,125 V)."
- note added: "AI1 — Druck 0–10 V"
- note added: "AI2 — Durchfluss 4–20 mA"
- note added: "AI3 — Wassertemp 4–20 mA"
- note added: "AI4 — Regentonne 4–20 mA"
- note added: "AI5 — Reserve"
- note added: "AI6 — Reserve"
- note added: "JP gesteckt: 4–20 mA → 150 Ω. JP offen: 0–10 V. PTC 50 mA in Speisung und Eingang, TVS SMAJ26A."
- note added: "MON_24V = 24 V / 11 (2,18 V), MON_5V = 5 V / 2 (2,5 V)."
- note added: "Versorgungsüberwachung"
- note removed: "ADC 1 (0x48: AI1–AI4) / ADC 2 (0x49: AI5, AI6, 24V, 5V)"
- note removed: "AI1 — Druck 0–10 V (JP gesteckt = 4–20 mA / 150 Ω, offen = 0–10 V)"
- note removed: "AI2 — Durchfluss 4–20 mA (JP gesteckt = 4–20 mA / 150 Ω, offen = 0–10 V)"
- note removed: "AI3 — Wassertemp 4–20 mA (JP gesteckt = 4–20 mA / 150 Ω, offen = 0–10 V)"
- note removed: "AI4 — Regentonne 4–20 mA (JP gesteckt = 4–20 mA / 150 Ω, offen = 0–10 V)"
- note removed: "AI5 — Reserve (JP gesteckt = 4–20 mA / 150 Ω, offen = 0–10 V)"
- note removed: "AI6 — Reserve (JP gesteckt = 4–20 mA / 150 Ω, offen = 0–10 V)"
- note removed: "Spannungsüberwachung"
- title: 6 × Universal-Analogeingang 0–10 V / 4–20 mA (Jumper) -> Analogeingänge 6 × 0–10 V / 4–20 mA
