File: hardware/kicad/analog_out.kicad_sch (KiCad schematic)
At the start: 31 parts, among them J13 AO1: I+ / GND, J14 AO2: I+ / GND, Q1 2N7002, Q2 MMBT2907A, Q3 BSP170P, Q4 MMBT2907A, Q5 BSP170P, U5 MCP4728-E/UN, U6 XTR111AIDGQR, U7 XTR111AIDGQR

Commit message: hardware: Rev 0.2 – ESP32-S3 (Steuerung) + M5Stack Stamp-P4 (App/HMI) statt CM5
CM5 entfernt. Neu: ESP32-S3-WROOM-1 für Regelung/I/O/V20, Stamp-P4 mit
LAN8720A-Ethernet und 7"-MIPI-DSI-Touch (FPC 15p), UART-Link mit Reset/Boot-
Steuerung des S3 durch den P4, 5V->3,3V-Wandler, USB-Werkbankversorgung.
I/O-Blätter unverändert. Netzliste geprüft (180 Netze, 0 Fehler).

Co-Authored-By: Claude Opus 5.5 <noreply@anthropic.com>
Claude-Session: https://claude.ai/code/session_019gH4tfEhDrFu8dTGZD88nH
Parts:
- removed C32: 100nF, Capacitor_SMD:C_0603_1608Metric, symbol Device:C
- removed C33: 10µF, Capacitor_SMD:C_0805_2012Metric, symbol Device:C
- removed C34, C37: 100nF/50V, Capacitor_SMD:C_0603_1608Metric, symbol Device:C
- removed C35, C38: 2.2nF, Capacitor_SMD:C_0603_1608Metric, symbol Device:C
- removed C36, C39: 10nF/50V, Capacitor_SMD:C_0603_1608Metric, symbol Device:C
- removed D11, D13: 1N4148W, Diode_SMD:D_SOD-123, symbol Diode:1N4148W
- removed D12, D14: SMAJ26A, Diode_SMD:D_SMA, symbol Diode:SMAJ26A
- removed J13: AO1: I+ / GND, TerminalBlock_Phoenix:TerminalBlock_Phoenix_PT-1,5-2-3.5-H_1x02_P3.50mm_Horizontal, symbol Connector:Screw_Terminal_01x02
- removed Q1: 2N7002, Package_TO_SOT_SMD:SOT-23, symbol Transistor_FET:2N7002
- removed Q2: MMBT2907A, Package_TO_SOT_SMD:SOT-23, symbol Transistor_BJT:MMBT3906
- removed Q3: BSP170P, Package_TO_SOT_SMD:SOT-223-3_TabPin2, symbol Device:Q_PMOS_GDS
- removed R44: 100, Resistor_SMD:R_0603_1608Metric, symbol Device:R
- removed R45: 100k, Resistor_SMD:R_0603_1608Metric, symbol Device:R
- removed R46: 10k, Resistor_SMD:R_0603_1608Metric, symbol Device:R
- removed R47, R50: 1.00k 0.1%, Resistor_SMD:R_0603_1608Metric, symbol Device:R
- removed R48, R49, R51, R52: 15, Resistor_SMD:R_0603_1608Metric, symbol Device:R
- removed U5: MCP4728-E/UN, Package_SO:MSOP-10_3x3mm_P0.5mm, symbol Analog_DAC:MCP4728
- removed U6, U7: XTR111AIDGQR, Package_SO:MSOP-10-1EP_3x3mm_P0.5mm_EP2.2x3.1mm_Mask1.83x1.89mm_ThermalVias, symbol Interface_CurrentLoop:XTR111AxDGQ
- added C45: 100nF, Capacitor_SMD:C_0603_1608Metric, symbol Device:C
- added C46: 10µF, Capacitor_SMD:C_0805_2012Metric, symbol Device:C
- added C47, C50: 100nF/50V, Capacitor_SMD:C_0603_1608Metric, symbol Device:C
- added C48, C51: 2.2nF, Capacitor_SMD:C_0603_1608Metric, symbol Device:C
- added C49, C52: 10nF/50V, Capacitor_SMD:C_0603_1608Metric, symbol Device:C
- added D12, D14: 1N4148W, Diode_SMD:D_SOD-123, symbol Diode:1N4148W
- added D13, D15: SMAJ26A, Diode_SMD:D_SMA, symbol Diode:SMAJ26A
- added J15: AO2: I+ / GND, TerminalBlock_Phoenix:TerminalBlock_Phoenix_PT-1,5-2-3.5-H_1x02_P3.50mm_Horizontal, symbol Connector:Screw_Terminal_01x02
- added Q3: 2N7002, Package_TO_SOT_SMD:SOT-23, symbol Transistor_FET:2N7002
- added Q6: MMBT2907A, Package_TO_SOT_SMD:SOT-23, symbol Transistor_BJT:MMBT3906
- added Q7: BSP170P, Package_TO_SOT_SMD:SOT-223-3_TabPin2, symbol Device:Q_PMOS_GDS
- added R59: 100, Resistor_SMD:R_0603_1608Metric, symbol Device:R
- added R60: 100k, Resistor_SMD:R_0603_1608Metric, symbol Device:R
- added R61: 10k, Resistor_SMD:R_0603_1608Metric, symbol Device:R
- added R62, R65: 1.00k 0.1%, Resistor_SMD:R_0603_1608Metric, symbol Device:R
- added R63, R64, R66, R67: 15, Resistor_SMD:R_0603_1608Metric, symbol Device:R
- added U10, U11: XTR111AIDGQR, Package_SO:MSOP-10-1EP_3x3mm_P0.5mm_EP2.2x3.1mm_Mask1.83x1.89mm_ThermalVias, symbol Interface_CurrentLoop:XTR111AxDGQ
- added U9: MCP4728-E/UN, Package_SO:MSOP-10_3x3mm_P0.5mm, symbol Analog_DAC:MCP4728
- J14: value AO2: I+ / GND -> AO1: I+ / GND
Connections:
- net +24V: now also C47.1, C50.1, D12.1 (K), D14.1 (K), U10.1 (VSP), U11.1 (VSP)
- net +3V3: now also C45.1, C46.1, R61.1, U9.1 (VDD)
- net AO1_D: now also Q5.2 (D), R64.1
- net AO1_IS: now also Q4.2 (E), R63.1, U10.2 (IS)
- net AO1_OUT: now also J14.1 (Pin_1), C49.1, D12.2 (A), D13.1 (A1), R64.2
- net AO1_REG: now also C48.1, U10.4 (REGS), U10.5 (REGF)
- net AO1_RSET: now also R62.1, U10.7 (SET)
- net AO1_S: now also Q4.1 (B), Q5.3 (S), R63.2
- net AO1_SET: now also U10.6 (VIN), U9.6 (VOUTA)
- net AO1_VG: now also Q4.3 (C), Q5.1 (G), U10.3 (VG)
- net AO2_D: now also Q7.2 (D), R67.1; no longer Q5.2 (D)
- net AO2_IS: now also Q6.2 (E), R66.1, U11.2 (IS); no longer Q4.2 (E)
- net AO2_OUT: now also C52.1, D14.2 (A), D15.1 (A1), J15.1 (Pin_1), R67.2; no longer J14.1 (Pin_1)
- net AO2_REG: now also C51.1, U11.4 (REGS), U11.5 (REGF)
- net AO2_RSET: now also R65.1, U11.7 (SET)
- net AO2_S: now also Q6.1 (B), Q7.3 (S), R66.2; no longer Q4.1 (B), Q5.3 (S)
- net AO2_SET: now also U11.6 (VIN), U9.7 (VOUTB)
- net AO2_VG: now also Q6.3 (C), Q7.1 (G), U11.3 (VG); no longer Q4.3 (C), Q5.1 (G)
- net AO_EN: now also R59.1
- net AO_EN_G: now also Q3.1 (G), R59.2, R60.1
- net AO_FAULT: now also R61.2, U10.8 (~{EF}), U11.8 (~{EF})
- net AO_OD: now also Q3.3 (D), U10.9 (OD), U11.9 (OD)
- net GND: now also C45.2, C46.2, C47.2, C48.2, C49.2, C50.2, C51.2, C52.2, D13.2 (A2), D15.2 (A2), J15.2 (Pin_2), Q3.2 (S), R60.2, R62.2, R65.2, U10.10 (GND), U10.11 (GND), U11.10 (GND), U11.11 (GND), U9.10 (VSS), U9.4 (~{LDAC})
- net I2C_SCL: now also U9.2 (SCL)
- net I2C_SDA: now also U9.3 (SDA)

Commit message: hardware: Schaltplan im Block-Stil wie pool-pcb
Neuer Generator tools/schblock.py: gestrichelte Funktionsblöcke mit Titel und
Notizen, echte Drähte (eigener Router), Power-Symbole am Pin bzw. als Schiene,
Global-Labels nur an Blockgrenzen. Netzliste weiterhin gegen die deklarierte
Absicht geprüft (180 Netze, 0 Fehler), PWR_FLAGs ergänzt.

Co-Authored-By: Claude Opus 5.5 <noreply@anthropic.com>
Claude-Session: https://claude.ai/code/session_019gH4tfEhDrFu8dTGZD88nH
Parts:
- removed C52: 10nF/50V, Capacitor_SMD:C_0603_1608Metric, symbol Device:C
- added C44: 100nF, Capacitor_SMD:C_0603_1608Metric, symbol Device:C
- C45: value 100nF -> 10µF; footprint Capacitor_SMD:C_0603_1608Metric -> Capacitor_SMD:C_0805_2012Metric
- C46: value 10µF -> 100nF/50V; footprint Capacitor_SMD:C_0805_2012Metric -> Capacitor_SMD:C_0603_1608Metric
- C47, C50: value 100nF/50V -> 2.2nF
- C48, C51: value 2.2nF -> 10nF/50V
- C49: value 10nF/50V -> 100nF/50V
- J14: value AO1: I+ / GND -> AO1
- J15: value AO2: I+ / GND -> AO2
Connections:
- net +24V: now also C46.1, C49.1; no longer C47.1, C50.1
- net +3V3: now also C44.1; no longer C46.1
- net GND: now also C44.2
- net AO1_D: no longer names the net of Q5.2 (D), R64.1
- net AO1_IS: no longer names the net of Q4.2 (E), R63.1, U10.2 (IS)
- net AO1_OUT: no longer names the net of D12.2 (A), D13.1 (A1), J14.1 (Pin_1), R64.2
- net AO1_OUT: now also C48.1; no longer C49.1
- net AO1_REG: no longer names the net of U10.4 (REGS), U10.5 (REGF)
- net AO1_REG: now also C47.1; no longer C48.1
- net AO1_RSET: no longer names the net of R62.1, U10.7 (SET)
- net AO1_S: no longer names the net of Q4.1 (B), Q5.3 (S), R63.2
- net AO1_VG: no longer names the net of Q4.3 (C), Q5.1 (G), U10.3 (VG)
- net AO2_D: no longer names the net of Q7.2 (D), R67.1
- net AO2_IS: no longer names the net of Q6.2 (E), R66.1, U11.2 (IS)
- net AO2_OUT: no longer names the net of D14.2 (A), D15.1 (A1), J15.1 (Pin_1), R67.2
- net AO2_OUT: now also C51.1
- net AO2_REG: no longer names the net of U11.4 (REGS), U11.5 (REGF)
- net AO2_REG: now also C50.1; no longer C51.1
- net AO2_RSET: no longer names the net of R65.1, U11.7 (SET)
- net AO2_S: no longer names the net of Q6.1 (B), Q7.3 (S), R66.2
- net AO2_VG: no longer names the net of Q6.3 (C), Q7.1 (G), U11.3 (VG)
- net AO_EN_G: no longer names the net of Q3.1 (G), R59.2, R60.1
Other:
- note added: "4 mA = Code 800, 20 mA = Code 4000."
- note added: "AO1 — Dosierpumpe (0…20,48 mA, Bürde ≤ 900 Ω)"
- note added: "AO2 — Reserve (0…20,48 mA, Bürde ≤ 900 Ω)"
- note added: "AO_EN LOW (Boot, Absturz) → OD = HIGH → beide Ausgänge 0 mA. AO_FAULT LOW = Drahtbruch / Bürde zu hoch."
- note added: "Ausgangsfreigabe & Fehlermeldung"
- note added: "DAC MCP4728 (I²C 0x60, int. Ref. 2,048 V)"
- note added: "PNP + 15 Ω begrenzt auf ≈ 37 mA. Diode gegen Überspannung an +24 V, TVS gegen GND."
- note removed: "AO1 — Dosierpumpe I = 10 · U_DAC / 1 kΩ (0…20,48 mA)"
- note removed: "AO2 — Reserve I = 10 · U_DAC / 1 kΩ (0…20,48 mA)"
- note removed: "DAC (I²C 0x60, interne Ref. 2,048 V) & Ausgangsfreigabe"
- title: 2 × Analogausgang 0/4–20 mA (Dosierpumpe + Reserve) -> Analogausgänge 2 × 0/4–20 mA
