File: hardware/kicad/ctrl_s3.kicad_sch (KiCad schematic)
At the start: 22 parts, among them J2 USB-C S3, J3 Erweiterung S3, Q1 2N7002, Q2 2N7002, SW1 RESET S3, SW2 BOOT S3, SW3 SERVICE, U4 ESP32-S3-WROOM-1-N16R8

Commit message: hardware: Schaltplan im Block-Stil wie pool-pcb
Neuer Generator tools/schblock.py: gestrichelte Funktionsblöcke mit Titel und
Notizen, echte Drähte (eigener Router), Power-Symbole am Pin bzw. als Schiene,
Global-Labels nur an Blockgrenzen. Netzliste weiterhin gegen die deklarierte
Absicht geprüft (180 Netze, 0 Fehler), PWR_FLAGs ergänzt.

Co-Authored-By: Claude Opus 5.5 <noreply@anthropic.com>
Claude-Session: https://claude.ai/code/session_019gH4tfEhDrFu8dTGZD88nH
Parts:
- C23: value 1µF -> 1µ
- R11: value 10k -> 100k
- R12: value 100k -> 10k
- SW1: value RESET S3 -> RESET
- SW2: value BOOT S3 -> BOOT
Connections:
- net +3V3: now also R12.1; no longer R11.1
- net GND: now also R11.2; no longer R12.2
- net P4_S3_RST: now also R11.1; no longer R12.1
- net S3_IO0: now also R12.2; no longer R11.2
- net STAT_LED_A: no longer names the net of D4.2 (A), R17.2
- net USB_S3_CC1: no longer names the net of J2.A5 (CC1), R14.1
- net USB_S3_CC2: no longer names the net of J2.B5 (CC2), R15.1
Other:
- note added: "Bedienung & Status"
- note added: "ESP32-S3-WROOM-1-N16R8"
- note added: "IO3/IO45/IO46 = Strapping, IO35–37 = Octal-PSRAM → frei. UART0 (RXD0/TXD0) = Link zum P4 und zugleich Flash-Port → P4 kann den S3 per OTA flashen."
- note added: "I²C-Pull-ups & Erweiterung"
- note added: "P4_S3_RST / P4_S3_BOOT = HIGH zieht EN bzw. IO0 auf GND."
- note added: "Reset / Boot (Taster + vom P4 steuerbar)"
- note added: "USB-C (Flashen, Konsole, Werkbank-Versorgung)"
- note removed: "Bedienung, LED, I²C-Pull-ups, Erweiterung"
- note removed: "ESP32-S3-WROOM-1-N16R8 (IO3/IO45/IO46 = Straps, IO35–37 = Octal-PSRAM → frei lassen)"
- note removed: "Reset / Boot (auch vom P4 aus steuerbar → P4 kann die Steuerung per OTA flashen)"
- note removed: "USB-C (S3 flashen / Konsole; versorgt die Platine auf der Werkbank ohne 230 V)"
- title: Steuerung: ESP32-S3-WROOM-1 (Regelung, I/O, V20, Sicherheit) -> Steuerung: ESP32-S3-WROOM-1
