File: hardware/kicad/hmi_p4.kicad_sch (KiCad schematic)
At the start: 42 parts, among them J4 Erweiterung P4, J5 HR911105A, J6 DSI 15p 1.0mm, J7 Display 5V, SW4 RESET P4, SW5 BOOT P4, U5 M5Stack Stamp-P4, U6 LAN8720A-CP, Y1 25MHz 18pF

Commit message: hardware: Schaltplan im Block-Stil wie pool-pcb
Neuer Generator tools/schblock.py: gestrichelte Funktionsblöcke mit Titel und
Notizen, echte Drähte (eigener Router), Power-Symbole am Pin bzw. als Schiene,
Global-Labels nur an Blockgrenzen. Netzliste weiterhin gegen die deklarierte
Absicht geprüft (180 Netze, 0 Fehler), PWR_FLAGs ergänzt.

Co-Authored-By: Claude Opus 5.5 <noreply@anthropic.com>
Claude-Session: https://claude.ai/code/session_019gH4tfEhDrFu8dTGZD88nH
Parts:
- removed C34: 22µF/16V, Capacitor_SMD:C_1210_3225Metric, symbol Device:C
- C26: value 10µF -> 10µ
- C27, C28: value 100nF -> 100n
- C29: value 100nF -> 1µ
- C30: value 1µF -> 470p
- C31: value 470pF -> 22p
- C32: value 22pF -> 22p
- C33: value 22pF -> 22µ/16V; footprint Capacitor_SMD:C_0603_1608Metric -> Capacitor_SMD:C_1210_3225Metric
- H1, H2, H3, H4: value Gehäuse M3 -> M3
- R27, R28, R29, R30: value 49.9 1% -> 49.9
- Y1: value 25MHz 18pF -> 25MHz
Connections:
- net +3V3: now also C28.1; no longer C29.1
- net ETH_AVDD: now also R27.1, R28.1, R29.1, R30.1; no longer C28.1, R27.2, R28.2, R29.2, R30.2
- net ETH_TXP: now also R27.2; no longer R27.1
- net RMII_CLK_P4: now also R23.1; no longer R23.2
- net DISP_5V: no longer names the net of F2.2, J7.1 (Pin_1)
- net DISP_5V: now also C33.1
- net ETH_LED1: no longer names the net of R32.1
- net ETH_LED1: now also R26.1, U6.2 (LED2/~{INTSEL}); no longer U6.3 (LED1/REGOFF)
- removed net ETH_LED2: R26.1, R31.1, U6.2 (LED2/~{INTSEL})
- net ETH_LEDG_A: no longer names the net of R31.2
- net ETH_LEDG_A: now also J5.12; no longer J5.9
- net ETH_LEDY_A: no longer names the net of R32.2
- net ETH_LEDY_A: now also J5.9; no longer J5.12
- net ETH_RBIAS: no longer names the net of R22.1, U6.24 (RBIAS)
- net ETH_REFCLK: no longer names the net of U6.14 (~{INT}/REFCLKO)
- net ETH_REFCLK: now also R23.2; no longer R23.1
- net ETH_RXN: no longer names the net of J5.6 (RD-), U6.22 (RXN)
- net ETH_RXN: now also R30.2; no longer R30.1
- net ETH_RXP: no longer names the net of J5.3 (RD+), U6.23 (RXP)
- net ETH_RXP: now also R29.2; no longer R29.1
- net ETH_TXN: no longer names the net of J5.2 (TD-), U6.20 (TXN)
- net ETH_TXN: now also R28.2; no longer R28.1
- net ETH_VDDCR: no longer names the net of C30.1, U6.6 (VDDCR)
- net ETH_VDDCR: now also C29.1; no longer C31.1
- net ETH_XI: no longer names the net of U6.5 (XTAL1/CLKIN), Y1.1
- net ETH_XI: now also C31.1; no longer C32.1
- net ETH_XO: no longer names the net of U6.4 (XTAL2), Y1.3
- net ETH_XO: now also C32.1; no longer C33.1
- net P4_LED_A: no longer names the net of D5.2 (A), R21.2
- new net: R31.1, U6.3 (LED1/REGOFF)
Other:
- note added: "7"-Display (MIPI-DSI 2-Lane, FPC 15-pol. 1,0 mm, Raspberry-Pi-Belegung)"
- note added: "BOOT P4 liegt auf G35 (= RMII_TXD1), nur beim Reset drücken."
- note added: "Bedienung, Link zum S3, Erweiterung"
- note added: "Ethernet 10/100 (LAN8720A, 25-MHz-Quarz, REFCLKO 50 MHz → P4)"
- note added: "M5Stack Stamp-P4 (ESP32-P4, 16 MB Flash, 32 MB PSRAM)"
- note added: "Modul wird aufgelötet (RMII + DSI nur an den Randpads oben). Eigener USB-C des Moduls = Flash/Konsole P4 → an den Platinenrand setzen."
- note added: "Touch-I²C über FPC (Pin 11/12). Display-Logik 3,3 V über Pin 15, Hintergrundbeleuchtung 5 V separat. DSI-Paare 100 Ω differentiell, so kurz wie möglich."
- note added: "nINTSEL = 0 (R an LED2) → Pin 14 liefert 50 MHz Referenztakt. PHY-Adresse 0. 4 × 49,9 Ω an ETH_AVDD (gefiltert über FB1), Mittelanzapfungen ebenfalls an ETH_AVDD."
- note removed: "7"-Display: MIPI-DSI 2-Lane, FPC 15-pol. 1,0 mm (Raspberry-Pi-Standard) + 5-V-Versorgung"
- note removed: "Ethernet-PHY LAN8720A (25-MHz-Quarz, REFCLKO 50 MHz → P4)"
- note removed: "M5Stack Stamp-P4 (ESP32-P4, 16 MB Flash, 32 MB PSRAM) — eigener USB-C am Platinenrand zugänglich"
- title: App/HMI: M5Stack Stamp-P4, Ethernet (LAN8720A), 7"-DSI-Touch -> App/HMI: Stamp-P4, Ethernet, 7"-Display
