File: hardware/kicad/io.kicad_sch (KiCad schematic)
At the start: 56 parts, among them J15 DI: 24V / DI1–DI4 / GND, J16 K1: NO / COM / NC, J17 K2: NO / COM / NC, J18 RS485: A(P+) / B(N-) / GND_ISO, J19 Lüfter 4-Pin, K1 34.51.7.024.0010, K2 34.51.7.024.0010, Q6 2N7002, Q7 2N7002, U10 74LVC1G07, U8 TLP293-4, U9 ADM2587EBRWZ

Commit message: hardware: Rev 0.2 – ESP32-S3 (Steuerung) + M5Stack Stamp-P4 (App/HMI) statt CM5
CM5 entfernt. Neu: ESP32-S3-WROOM-1 für Regelung/I/O/V20, Stamp-P4 mit
LAN8720A-Ethernet und 7"-MIPI-DSI-Touch (FPC 15p), UART-Link mit Reset/Boot-
Steuerung des S3 durch den P4, 5V->3,3V-Wandler, USB-Werkbankversorgung.
I/O-Blätter unverändert. Netzliste geprüft (180 Netze, 0 Fehler).

Co-Authored-By: Claude Opus 5.5 <noreply@anthropic.com>
Claude-Session: https://claude.ai/code/session_019gH4tfEhDrFu8dTGZD88nH
Parts:
- removed C40, C41, C42, C43: 10nF, Capacitor_SMD:C_0603_1608Metric, symbol Device:C
- removed C44, C47: 10µF, Capacitor_SMD:C_0805_2012Metric, symbol Device:C
- removed C45, C46, C48, C49: 100nF, Capacitor_SMD:C_0603_1608Metric, symbol Device:C
- removed D15, D17, D19, D21: BZT52C9V1, Diode_SMD:D_SOD-123, symbol Device:D_Zener
- removed D16, D18, D20, D22, D25: 1N4148W, Diode_SMD:D_SOD-123, symbol Diode:1N4148W
- removed D24: rot K1, LED_SMD:LED_0603_1608Metric, symbol Device:LED
- removed D26: rot K2, LED_SMD:LED_0603_1608Metric, symbol Device:LED
- removed D27: SMAJ15CA, Diode_SMD:D_SMA, symbol Diode:SMAJ15CA
- removed F14: 200mA hold, Fuse:Fuse_1206_3216Metric, symbol Device:Polyfuse
- removed J15: DI: 24V / DI1–DI4 / GND, TerminalBlock_Phoenix:TerminalBlock_Phoenix_PT-1,5-6-3.5-H_1x06_P3.50mm_Horizontal, symbol Connector:Screw_Terminal_01x06
- removed J16: K1: NO / COM / NC, TerminalBlock_Phoenix:TerminalBlock_Phoenix_MKDS-1,5-3-5.08_1x03_P5.08mm_Horizontal, symbol Connector:Screw_Terminal_01x03
- removed J19: Lüfter 4-Pin, Connector:FanPinHeader_1x04_P2.54mm_Vertical, symbol Connector_Generic:Conn_01x04
- removed JP8: 120Ω Abschluss, Connector_PinHeader_2.54mm:PinHeader_1x02_P2.54mm_Vertical, symbol Jumper:Jumper_2_Open
- removed Q6, Q7: 2N7002, Package_TO_SOT_SMD:SOT-23, symbol Transistor_FET:2N7002
- removed R53, R55, R57, R59: 3.3k, Resistor_SMD:R_1206_3216Metric, symbol Device:R
- removed R54, R56, R58, R60, R67: 10k, Resistor_SMD:R_0603_1608Metric, symbol Device:R
- removed R61, R64: 100, Resistor_SMD:R_0603_1608Metric, symbol Device:R
- removed R62, R65: 100k, Resistor_SMD:R_0603_1608Metric, symbol Device:R
- removed R63, R66: 4.7k, Resistor_SMD:R_0603_1608Metric, symbol Device:R
- removed U10: 74LVC1G07, Package_TO_SOT_SMD:SOT-23-5, symbol 74xGxx:74LVC1G07
- removed U8: TLP293-4, Package_SO:SOIC-16_4.55x10.3mm_P1.27mm, symbol Isolator:TLP293-4
- removed U9: ADM2587EBRWZ, Package_SO:SOIC-20W_7.5x12.8mm_P1.27mm, symbol Interface_UART:ADM2587E
- added C53, C54, C55, C56: 10nF, Capacitor_SMD:C_0603_1608Metric, symbol Device:C
- added C57, C60: 10µF, Capacitor_SMD:C_0805_2012Metric, symbol Device:C
- added C58, C59, C61, C62: 100nF, Capacitor_SMD:C_0603_1608Metric, symbol Device:C
- added D16, D18, D20, D22: BZT52C9V1, Diode_SMD:D_SOD-123, symbol Device:D_Zener
- added D17, D19, D21, D24, D26: 1N4148W, Diode_SMD:D_SOD-123, symbol Diode:1N4148W
- added D25: rot K1, LED_SMD:LED_0603_1608Metric, symbol Device:LED
- added D27: rot K2, LED_SMD:LED_0603_1608Metric, symbol Device:LED
- added D29: SMAJ15CA, Diode_SMD:D_SMA, symbol Diode:SMAJ15CA
- added F15: 200mA hold, Fuse:Fuse_1206_3216Metric, symbol Device:Polyfuse
- added J16: DI: 24V / DI1–DI4 / GND, TerminalBlock_Phoenix:TerminalBlock_Phoenix_PT-1,5-6-3.5-H_1x06_P3.50mm_Horizontal, symbol Connector:Screw_Terminal_01x06
- added J19: RS485: A(P+) / B(N-) / GND_ISO, TerminalBlock_Phoenix:TerminalBlock_Phoenix_PT-1,5-3-3.5-H_1x03_P3.50mm_Horizontal, symbol Connector:Screw_Terminal_01x03
- added J20: Lüfter 4-Pin, Connector:FanPinHeader_1x04_P2.54mm_Vertical, symbol Connector_Generic:Conn_01x04
- added JP7: 120Ω Abschluss, Connector_PinHeader_2.54mm:PinHeader_1x02_P2.54mm_Vertical, symbol Jumper:Jumper_2_Open
- added Q8, Q9: 2N7002, Package_TO_SOT_SMD:SOT-23, symbol Transistor_FET:2N7002
- added R71, R73, R75, R82, R84, R85: 10k, Resistor_SMD:R_0603_1608Metric, symbol Device:R
- added R72, R74: 3.3k, Resistor_SMD:R_1206_3216Metric, symbol Device:R
- added R76, R79: 100, Resistor_SMD:R_0603_1608Metric, symbol Device:R
- added R77, R80: 100k, Resistor_SMD:R_0603_1608Metric, symbol Device:R
- added R78, R81: 4.7k, Resistor_SMD:R_0603_1608Metric, symbol Device:R
- added R83: 120, Resistor_SMD:R_1206_3216Metric, symbol Device:R
- added U12: TLP293-4, Package_SO:SOIC-16_4.55x10.3mm_P1.27mm, symbol Isolator:TLP293-4
- added U13: ADM2587EBRWZ, Package_SO:SOIC-20W_7.5x12.8mm_P1.27mm, symbol Interface_UART:ADM2587E
- added U14: 74LVC1G07, Package_TO_SOT_SMD:SOT-23-5, symbol 74xGxx:74LVC1G07
- J17: value K2: NO / COM / NC -> K1: NO / COM / NC
- J18: value RS485: A(P+) / B(N-) / GND_ISO -> K2: NO / COM / NC; footprint TerminalBlock_Phoenix:TerminalBlock_Phoenix_PT-1,5-3-3.5-H_1x03_P3.50mm_Horizontal -> TerminalBlock_Phoenix:TerminalBlock_Phoenix_MKDS-1,5-3-5.08_1x03_P5.08mm_Horizontal
- R68: value 120 -> 3.3k
- R70: value 10k -> 3.3k; footprint Resistor_SMD:R_0603_1608Metric -> Resistor_SMD:R_1206_3216Metric
Connections:
- net +12V: now also J20.2 (Pin_2)
- net +24V: now also D24.1 (K), D26.1 (K), F15.1, R78.1, R81.1; no longer D23.1 (K)
- net +3V3: now also C57.1, C58.1, C59.1, C62.1, R71.1, R73.1, R75.1, R84.1, U13.2 (VCC), U13.8 (VCC), U14.5 (VCC)
- net DI1: now also R69.2, C53.1, U12.16
- net DI1_A: now also R68.2, D17.1 (K), U12.1
- net DI1_IN: now also D16.1 (K), J16.2 (Pin_2)
- net DI1_Z: now also R68.1, D16.2 (A)
- net DI2: now also C54.1, R71.2, U12.14
- net DI2_A: now also R70.2, D19.1 (K), U12.3
- net DI2_IN: now also D18.1 (K), J16.3 (Pin_3)
- net DI2_Z: now also R70.1, D18.2 (A)
- net DI3: now also C55.1, R73.2, U12.12
- net DI3_A: now also D21.1 (K), R72.2, U12.5
- net DI3_IN: now also D20.1 (K), J16.4 (Pin_4)
- net DI3_Z: now also D20.2 (A), R72.1
- net DI4: now also C56.1, R75.2, U12.10
- net DI4_A: now also D23.1 (K), R74.2, U12.7
- net DI4_IN: now also D22.1 (K), J16.5 (Pin_5)
- net DI4_Z: now also D22.2 (A), R74.1
- net DI_24V: now also F15.2, J16.1 (Pin_1)
- net FAN_PWM: now also U14.2
- net FAN_PWM_OD: now also J20.4 (Pin_4), U14.4
- net FAN_TACH: now also R85.2; no longer R70.2
- net FAN_TACH_IN: now also J20.3 (Pin_3), R84.2, R85.1; no longer R69.2, R70.1
- net GND: now also D23.2 (A), C53.2, C54.2, C55.2, C56.2, C57.2, C58.2, C59.2, C62.2, D17.2 (A), D19.2 (A), D21.2 (A), J16.6 (Pin_6), J20.1 (Pin_1), Q8.2 (S), Q9.2 (S), R77.2, R80.2, R82.2, U12.11, U12.13, U12.15, U12.2, U12.4, U12.6, U12.8, U12.9, U13.1 (GND1), U13.10 (GND1), U13.3 (GND1), U13.9 (GND1), U14.3 (GND)
- net GND_ISO: now also C60.2, C61.2, D29.2 (A2), J19.3 (Pin_3), U13.11 (GND2), U13.14 (GND2), U13.16 (GND2), U13.20 (GND2); no longer J18.3 (Pin_3)
- net RELAY1: now also R76.1
- net RELAY2: now also R79.1
- net RL1_COIL: now also D24.2 (A), D25.1 (K), Q8.3 (D); no longer D23.2 (A)
- net RL1_COM: now also J17.2 (Pin_2)
- net RL1_G: now also Q8.1 (G), R76.2, R77.1
- net RL1_LED: now also D25.2 (A), R78.2
- net RL1_NC: now also J17.3 (Pin_3)
- net RL1_NO: now also J17.1 (Pin_1)
- net RL2_COIL: now also D26.2 (A), D27.1 (K), Q9.3 (D)
- net RL2_COM: now also J18.2 (Pin_2); no longer J17.2 (Pin_2)
- net RL2_G: now also Q9.1 (G), R79.2, R80.1
- net RL2_LED: now also D27.2 (A), R81.2
- net RL2_NC: now also J18.3 (Pin_3); no longer J17.3 (Pin_3)
- net RL2_NO: now also J18.1 (Pin_1); no longer J17.1 (Pin_1)
- net RS485_A: now also D28.1 (A1), J19.1 (Pin_1), R83.1, U13.13 (Y), U13.18 (A); no longer J18.1 (Pin_1), R68.1
- net RS485_B: now also D29.1 (A1), J19.2 (Pin_2), JP7.2 (B), U13.15 (Z), U13.17 (B); no longer D28.1 (A1), J18.2 (Pin_2)
- net RS485_DE: now also R82.1, U13.5 (~{RE}), U13.6 (DE)
- net RS485_RX: now also U13.4 (RxD)
- net RS485_T: now also JP7.1 (A), R83.2; no longer R68.2
- net RS485_TX: now also U13.7 (TxD)
- net VISO: now also C60.1, C61.1, U13.12 (Visoout), U13.19 (Visoin)

Commit message: hardware: Schaltplan im Block-Stil wie pool-pcb
Neuer Generator tools/schblock.py: gestrichelte Funktionsblöcke mit Titel und
Notizen, echte Drähte (eigener Router), Power-Symbole am Pin bzw. als Schiene,
Global-Labels nur an Blockgrenzen. Netzliste weiterhin gegen die deklarierte
Absicht geprüft (180 Netze, 0 Fehler), PWR_FLAGs ergänzt.

Co-Authored-By: Claude Opus 5.5 <noreply@anthropic.com>
Claude-Session: https://claude.ai/code/session_019gH4tfEhDrFu8dTGZD88nH
Parts:
- removed C62: 100nF, Capacitor_SMD:C_0603_1608Metric, symbol Device:C
- added C52: 10nF, Capacitor_SMD:C_0603_1608Metric, symbol Device:C
- C56: value 10nF -> 10µF; footprint Capacitor_SMD:C_0603_1608Metric -> Capacitor_SMD:C_0805_2012Metric
- C57, C60: value 10µF -> 100nF; footprint Capacitor_SMD:C_0805_2012Metric -> Capacitor_SMD:C_0603_1608Metric
- C59: value 100nF -> 10µF; footprint Capacitor_SMD:C_0603_1608Metric -> Capacitor_SMD:C_0805_2012Metric
- C61: value 100nF -> 100n
- F15: value 200mA hold -> 200mA
- J16: value DI: 24V / DI1–DI4 / GND -> DI
- J17: value K1: NO / COM / NC -> K1
- J18: value K2: NO / COM / NC -> K2
- J19: value RS485: A(P+) / B(N-) / GND_ISO -> RS485
- JP7: value 120Ω Abschluss -> 120Ω
Connections:
- net +3V3: now also C56.1, C61.1; no longer C59.1
- net DI1: now also C52.1; no longer C53.1
- net DI2: now also C53.1; no longer C54.1
- net DI3: now also C54.1; no longer C55.1
- net DI4: now also C55.1; no longer C56.1
- net FAN_TACH: now also R85.1; no longer R85.2
- net FAN_TACH_IN: now also R85.2; no longer R85.1
- net GND: now also C61.2, C52.2; no longer C59.2
- net GND_ISO: now also C59.2; no longer C61.2
- net VISO: now also C59.1; no longer C61.1
- net DI1_A: no longer names the net of D17.1 (K), R68.2, U12.1
- net DI1_IN: no longer names the net of D16.1 (K), J16.2 (Pin_2)
- net DI1_Z: no longer names the net of D16.2 (A), R68.1
- net DI2_A: no longer names the net of D19.1 (K), R70.2, U12.3
- net DI2_IN: no longer names the net of D18.1 (K), J16.3 (Pin_3)
- net DI2_Z: no longer names the net of D18.2 (A), R70.1
- net DI3_A: no longer names the net of D21.1 (K), R72.2, U12.5
- net DI3_IN: no longer names the net of D20.1 (K), J16.4 (Pin_4)
- net DI3_Z: no longer names the net of D20.2 (A), R72.1
- net DI4_A: no longer names the net of D23.1 (K), R74.2, U12.7
- net DI4_IN: no longer names the net of D22.1 (K), J16.5 (Pin_5)
- net DI4_Z: no longer names the net of D22.2 (A), R74.1
- net DI_24V: no longer names the net of F15.2, J16.1 (Pin_1)
- net FAN_PWM_OD: no longer names the net of J20.4 (Pin_4), U14.4
- net RL1_COM: no longer names the net of J17.2 (Pin_2), K1.11
- net RL1_G: no longer names the net of Q8.1 (G), R76.2, R77.1
- net RL1_LED: no longer names the net of D25.2 (A), R78.2
- net RL1_NC: no longer names the net of J17.3 (Pin_3), K1.12
- net RL1_NO: no longer names the net of J17.1 (Pin_1), K1.14
- net RL2_COM: no longer names the net of J18.2 (Pin_2), K2.11
- net RL2_G: no longer names the net of Q9.1 (G), R79.2, R80.1
- net RL2_LED: no longer names the net of D27.2 (A), R81.2
- net RL2_NC: no longer names the net of J18.3 (Pin_3), K2.12
- net RL2_NO: no longer names the net of J18.1 (Pin_1), K2.14
- net RS485_A: no longer names the net of D28.1 (A1), J19.1 (Pin_1), R83.1, U13.13 (Y), U13.18 (A)
- net RS485_B: no longer names the net of D29.1 (A1), J19.2 (Pin_2), JP7.2 (B), U13.15 (Z), U13.17 (B)
- net RS485_T: no longer names the net of JP7.1 (A), R83.2
Other:
- note added: "74LVC1G07 Open-Drain: LOW = Lüfter langsam, offen = Lüfter-interner Pull-up → voll. Tacho mit Pull-up auf 3,3 V und 10k Serienwiderstand."
- note added: "DE + /RE gemeinsam (RTS/GPIO16), 10k Pull-down = Empfang. 120 Ω per Jumper. Klemme: A = P+, B = N−, GND_ISO an V20-Bezugspotenzial."
- note added: "Digitaleingänge 24 V (aktiv = GPIO LOW)"
- note added: "Gehäuselüfter 12 V (4-Pin-PWM 25 kHz, Tacho)"
- note added: "RS485 isoliert → V20 (Modbus RTU, Halbduplex)"
- note added: "Schaltschwelle ≈ 12 V (Z-Diode 9,1 V + LED). PTC 200 mA schützt die DI-Speisung."
- note removed: "Digitaleingänge 24 V (Schaltschwelle ≈ 12 V, aktiv = GPIO LOW)"
- note removed: "Gehäuselüfter 12 V, 4-Pin-PWM (GPIO18, 25 kHz) + Tacho (GPIO23)"
- note removed: "RS485 isoliert → V20 (Modbus RTU, Halbduplex, DE über RTS/GPIO17)"
- title: Digitaleingänge, Relais, RS485 (V20), Lüfter -> Digitaleingänge, Relais, RS485, Lüfter
