File: hardware/kicad/power.kicad_sch (KiCad schematic)
At the start: 35 parts, among them J1 230V L/N, U1 LMR33630ADDA, U2 LMR33630ADDA

Commit message: hardware: Rev 0.2 – ESP32-S3 (Steuerung) + M5Stack Stamp-P4 (App/HMI) statt CM5
CM5 entfernt. Neu: ESP32-S3-WROOM-1 für Regelung/I/O/V20, Stamp-P4 mit
LAN8720A-Ethernet und 7"-MIPI-DSI-Touch (FPC 15p), UART-Link mit Reset/Boot-
Steuerung des S3 durch den P4, 5V->3,3V-Wandler, USB-Werkbankversorgung.
I/O-Blätter unverändert. Netzliste geprüft (180 Netze, 0 Fehler).

Co-Authored-By: Claude Opus 5.5 <noreply@anthropic.com>
Claude-Session: https://claude.ai/code/session_019gH4tfEhDrFu8dTGZD88nH
Parts:
- removed D2: grün PWR, LED_SMD:LED_0603_1608Metric, symbol Device:LED
- removed U2: LMR33630ADDA, Package_SO:Texas_HSOP-8-1EP_3.9x4.9mm_P1.27mm_ThermalVias, symbol Regulator_Switching:LMR33630ADDA
- added C17: 100nF, Capacitor_SMD:C_0603_1608Metric, symbol Device:C
- added C18: 1µF, Capacitor_SMD:C_0603_1608Metric, symbol Device:C
- added C19, C20: 22µF/25V, Capacitor_SMD:C_1210_3225Metric, symbol Device:C
- added D2: SS14, Diode_SMD:D_SMA, symbol Diode:SS14
- added D3: grün PWR, LED_SMD:LED_0603_1608Metric, symbol Device:LED
- added L3: 22µH, Inductor_SMD:L_Bourns_SRP7028A_7.3x6.6mm, symbol Device:L
- added U2: AP63203WU-7, Package_TO_SOT_SMD:TSOT-23-6, symbol Regulator_Switching:AP63203WU
- added U3: LMR33630ADDA, Package_SO:Texas_HSOP-8-1EP_3.9x4.9mm_P1.27mm_ThermalVias, symbol Regulator_Switching:LMR33630ADDA
- C10: value 10µF/50V -> 10µF/16V; footprint Capacitor_SMD:C_1210_3225Metric -> Capacitor_SMD:C_0805_2012Metric
- C11: value 10µF/50V -> 100nF; footprint Capacitor_SMD:C_1210_3225Metric -> Capacitor_SMD:C_0603_1608Metric
- C12: value 100nF/50V -> 22µF/10V; footprint Capacitor_SMD:C_0603_1608Metric -> Capacitor_SMD:C_1210_3225Metric
- C13: value 100nF -> 22µF/10V; footprint Capacitor_SMD:C_0603_1608Metric -> Capacitor_SMD:C_1210_3225Metric
- C14: value 1µF -> 10µF/50V; footprint Capacitor_SMD:C_0603_1608Metric -> Capacitor_SMD:C_1210_3225Metric
- C15: value 22µF/25V -> 10µF/50V
- C16: value 22µF/25V -> 100nF/50V; footprint Capacitor_SMD:C_1210_3225Metric -> Capacitor_SMD:C_0603_1608Metric
- L2: value 22µH -> 4.7µH; footprint Inductor_SMD:L_Bourns_SRP7028A_7.3x6.6mm -> Inductor_SMD:L_Bourns-SRN6028; MPN Bourns SRP7028A-220M -> Bourns SRN6028-4R7M
Connections:
- net +12V: now also C19.1, C20.1, L3.2; no longer C15.1, C16.1, L2.2
- net +24V: now also C14.1, C15.1, C16.1, U3.2 (VIN); no longer C10.1, C11.1, C12.1
- net +5V: now also C10.1, D2.1 (K), U2.2 (EN), U2.3 (IN)
- net BUCK12_BOOT: now also C17.1, U3.7 (BOOT); no longer C13.1
- net BUCK12_EN: now also U3.3 (EN)
- net BUCK12_FB: now also U3.5 (FB)
- net BUCK12_SW: now also C17.2, L3.1, U3.8 (SW); no longer C13.2, L2.1
- net BUCK12_VCC: now also C18.1, U3.6 (VCC); no longer C14.1
- net GND: now also C13.2, C18.2, C19.2, C20.2, D3.1 (K), U2.4 (GND), U3.1 (GND), U3.9 (GND); no longer C11.2
- net PWR_LED_A: now also D3.2 (A)
- new net +3V3: C12.1, C13.1, L2.2, U2.1 (FB)
- new net BUCK3_BST: C11.1, U2.6 (BST)
- new net BUCK3_SW: C11.2, L2.1, U2.5 (SW)
- new net USB_S3_VBUS: D2.2 (A)
Other:
- note added: "24 V → 5 V / 3 A (Stamp-P4 + 7"-Display)"
- note added: "5 V → 3,3 V / 2 A (ESP32-S3, ADC/DAC, RS485, PHY) + USB-Versorgung für Werkbank"
- note removed: "24 V → 5 V / 3 A (CM5)"
- title: Stromversorgung 230 V → 24 V / 12 V / 5 V -> Stromversorgung 230 V → 24 V / 12 V / 5 V / 3,3 V

Commit message: hardware: Schaltplan im Block-Stil wie pool-pcb
Neuer Generator tools/schblock.py: gestrichelte Funktionsblöcke mit Titel und
Notizen, echte Drähte (eigener Router), Power-Symbole am Pin bzw. als Schiene,
Global-Labels nur an Blockgrenzen. Netzliste weiterhin gegen die deklarierte
Absicht geprüft (180 Netze, 0 Fehler), PWR_FLAGs ergänzt.

Co-Authored-By: Claude Opus 5.5 <noreply@anthropic.com>
Claude-Session: https://claude.ai/code/session_019gH4tfEhDrFu8dTGZD88nH
Parts:
- removed U2: AP63203WU-7, Package_TO_SOT_SMD:TSOT-23-6, symbol Regulator_Switching:AP63203WU
- removed U3: LMR33630ADDA, Package_SO:Texas_HSOP-8-1EP_3.9x4.9mm_P1.27mm_ThermalVias, symbol Regulator_Switching:LMR33630ADDA
- added U2: LMR33630ADDA, Package_SO:Texas_HSOP-8-1EP_3.9x4.9mm_P1.27mm_ThermalVias, symbol Regulator_Switching:LMR33630ADDA
- added U3: AP63203WU-7, Package_TO_SOT_SMD:TSOT-23-6, symbol Regulator_Switching:AP63203WU
- C10: value 10µF/16V -> 10µ/50V; footprint Capacitor_SMD:C_0805_2012Metric -> Capacitor_SMD:C_1210_3225Metric
- C11: value 100nF -> 10µ/50V; footprint Capacitor_SMD:C_0603_1608Metric -> Capacitor_SMD:C_1210_3225Metric
- C12: value 22µF/10V -> 100n/50V; footprint Capacitor_SMD:C_1210_3225Metric -> Capacitor_SMD:C_0603_1608Metric
- C13: value 22µF/10V -> 1µ; footprint Capacitor_SMD:C_1210_3225Metric -> Capacitor_SMD:C_0603_1608Metric
- C14: value 10µF/50V -> 100nF; footprint Capacitor_SMD:C_1210_3225Metric -> Capacitor_SMD:C_0603_1608Metric
- C15: value 10µF/50V -> 22µ/25V
- C16: value 100nF/50V -> 22µ/25V; footprint Capacitor_SMD:C_0603_1608Metric -> Capacitor_SMD:C_1210_3225Metric
- C17: value 100nF -> 10µF/16V; footprint Capacitor_SMD:C_0603_1608Metric -> Capacitor_SMD:C_0805_2012Metric
- C18, C6: value 1µF -> 100nF
- C19, C20: value 22µF/25V -> 22µF/10V
- C2, C3: value 10µF/50V -> 10µ/50V
- C4: value 100nF/50V -> 100n/50V
- C5: value 100nF -> 1µ
- C7, C8, C9: value 22µF/16V -> 22µ/16V
- F1: value T2A 250V 5x20 -> T2A 250V
- L2: value 4.7µH -> 22µH; footprint Inductor_SMD:L_Bourns-SRN6028 -> Inductor_SMD:L_Bourns_SRP7028A_7.3x6.6mm; MPN Bourns SRN6028-4R7M -> Bourns SRP7028A-220M
- L3: value 22µH -> 4.7µH; footprint Inductor_SMD:L_Bourns_SRP7028A_7.3x6.6mm -> Inductor_SMD:L_Bourns-SRN6028; MPN Bourns SRP7028A-220M -> Bourns SRN6028-4R7M
Connections:
- net BUCK12_BOOT is gone; now on net +5V: C17.1
- net BUCK3_BST is gone; now on net +24V: C11.1
- net +12V: now also C15.1, C16.1, L2.2; no longer C19.1, C20.1, L3.2
- net +24V: now also C10.1, C12.1, U2.2 (VIN); no longer C14.1, C15.1, C16.1
- net +3V3: now also C19.1, C20.1, L3.2, U3.1 (FB); no longer C12.1, C13.1, L2.2
- net +5V: now also U3.2 (EN), U3.3 (IN); no longer C10.1
- net GND: now also C11.2, C17.2, C5.2, U2.1 (GND), U2.9 (GND), U3.4 (GND); no longer C14.2, C18.2, C6.2
- net AC_L_IN: no longer names the net of F1.1, J1.1 (Pin_1)
- net BUCK12_EN: no longer names the net of R5.2, R6.1
- net BUCK12_EN: now also U2.3 (EN)
- net BUCK12_FB: no longer names the net of R7.2, R8.1
- net BUCK12_FB: now also U2.5 (FB)
- net BUCK12_SW: no longer names the net of L3.1
- net BUCK12_SW: now also C18.2, U3.5 (SW); no longer C17.2
- net BUCK12_VCC: no longer names the net of C18.1
- net BUCK12_VCC: now also U3.6 (BST)
- net BUCK3_SW: no longer names the net of L2.1
- net BUCK3_SW: now also C14.2, U2.8 (SW); no longer C11.2
- net BUCK5_BOOT: no longer names the net of U1.7 (BOOT)
- net BUCK5_BOOT: now also C6.1; no longer C5.1
- net BUCK5_EN: no longer names the net of R1.2, R2.1, U1.3 (EN)
- net BUCK5_FB: no longer names the net of R3.2, R4.1, U1.5 (FB)
- net BUCK5_SW: no longer names the net of L1.1, U1.8 (SW)
- net BUCK5_SW: now also C6.2; no longer C5.2
- net BUCK5_VCC: no longer names the net of U1.6 (VCC)
- net BUCK5_VCC: now also C5.1; no longer C6.1
- net PWR_LED_A: no longer names the net of D3.2 (A), R9.2
- new net: C13.1, U2.6 (VCC)
- new net: C14.1, U2.7 (BOOT)
Other:
- note added: "24 V → 12 V (Gehäuselüfter)"
- note added: "24-V-Schiene"
- note added: "5 V → 3,3 V / 2 A"
- note added: "AP63203 (Festspannung 3,3 V) für ESP32-S3, ADS1115, MCP4728, ADM2587E, LAN8720A. D2 SS14: USB-C des S3 versorgt die Platine auf der Werkbank (ohne 230 V)."
- note added: "Betriebsanzeige & Power-Flags"
- note added: "C1 Pufferung, D1 SMAJ30A gegen Überspannung auf 24 V."
- note added: "F1 T2A träge (5×20) vor dem Netzteil, RV1 275 VAC gegen Netzspitzen. Netzbereich: ≥ 6 mm Kriechstrecke + Frässchlitz zur Kleinspannung."
- note added: "LMR33630 400 kHz. U = 1 V · (1 + 100k / 24,9k) = 5,0 V. EN-Teiler: Einschalten ab ≈ 11 V."
- note added: "Netzeingang 230 V AC"
- note added: "Netzteil 24 V / 30 W"
- note added: "U = 1 V · (1 + 100k / 9,09k) = 12,0 V."
- note removed: "230 V AC Eingang (Netzbereich — Abstand ≥ 6 mm + Frässchlitz zur Niederspannung)"
- note removed: "24 V Schiene"
- note removed: "24 V → 12 V (Lüfter)"
- note removed: "5 V → 3,3 V / 2 A (ESP32-S3, ADC/DAC, RS485, PHY) + USB-Versorgung für Werkbank"
- note removed: "Anzeige & Power-Flags"
- title: Stromversorgung 230 V → 24 V / 12 V / 5 V / 3,3 V -> Stromversorgung 230 V / 24 V / 12 V / 5 V / 3,3 V
